File: electronics/breakup board/break-up board.kicad_pcb (KiCad board)
At the start: 2 copper layers, 0 parts

Commit message: 
Parts:
- added U1: CONN24, HEADER_2x12, F.Cu at (231.1, 129.5)
- added U2: CONN24, connect24, F.Cu at (237.5, 146.1)
Routing:
- net N-0000023: track 0.00 -> 82.5 mm
- net N-0000016: track 0.00 -> 77.8 mm
- net N-0000010: track 0.00 -> 71.2 mm
- net N-0000012: track 0.00 -> 67.2 mm
- net N-000003: track 0.00 -> 59.9 mm
- net N-0000019: track 0.00 -> 50.0 mm
- net N-000005: track 0.00 -> 49.0 mm
- net N-0000015: track 0.00 -> 37.0 mm
- net N-000007: track 0.00 -> 35.6 mm
- net N-000004: track 0.00 -> 21.0 mm
- net N-000008: track 0.00 -> 20.5 mm
- net N-000006: track 0.00 -> 20.4 mm
- net N-000001: track 0.00 -> 19.8 mm
- net N-0000013: track 0.00 -> 19.7 mm
- net N-000002: track 0.00 -> 19.7 mm
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Other:
- net class Default: clearance 0.254 -> 0.2032; trace_width 0.254 -> 0.2032
- rule trace_clearance: 0.254 -> 0.2032
- rule trace_min: 0.254 -> 0.2032
- rule via_min_size: 0.889 -> 0.2032
